File: einkpmic.sch (KiCad schematic (older format))
At the start: 29 parts

Commit message: update sch
Parts:
- added C38: 10uF/6.3V, symbol C_Small
- added C42, C45, C?: 4.7uF/50V, symbol C_Small
- added R59, R63, R66, R67, R?, SH35, SH38, SH39: 0/DNP, symbol R_Small
- added R?: 45.3K, symbol R_Small
Connections:
- net labels added: -1V25(EINK), E_PMIC_PWR0, I2C1_SCL, I2C1_SDA, PMICB_VPOS, PMIC_PGOOD
- wire segments 91 -> 130

Commit message: update sch
Parts:
- added C28, C34: 0.01uF/50V, symbol C_Small
- added C30, C35: 2.2uF/50V, symbol C_Small
- added C36, C37: 4.7uF/50V, symbol C_Small
- added D10, D8, D9, D? (x2): MBR130LSFT1G, symbol D_Schottky_Small
- added L4: 4.7uH, symbol L_Small
- added R253, R39, R49, SH37: 0/DNP, symbol R_Small
- added R42, R47: 1M, symbol R_Small
- added R43: 45.3K/DNP, symbol R_Small
- added R44: 47.5K, symbol R_Small
- added R46: 53.6K, symbol R_Small
- added R53: 330K, symbol R_Small
Connections:
- net labels added: +22V(EINK), -20V(EINK)
- wire segments 130 -> 193

Commit message: update sch
Parts:
- R45: renamed from R?; value 45.3K -> 100K
- gave numbers to parts that had none: 6

Commit message: update sch
Parts:
- C23: value 10uF/6.3V -> 4.7uF/50V
- C41: value 4.7uF/50V -> 10uF/6.3V
Connections:
- net labels added: PMICB_VSOURCE
- wire segments 193 -> 195
Other:
- moved on the sheet: C27, R36
Changed lines of the file:
@@
 LIBS:valves
 LIBS:einkpmic
+LIBS:einkpmic-cache
 EELAYER 25 0
 EELAYER END
@@
 P 4600 1500
 F 0 "C23" H 4610 1570 50  0000 L CNN
-F 1 "10uF/6.3V" H 4610 1420 50  0000 L CNN
+F 1 "4.7uF/50V" H 4610 1420 50  0000 L CNN
 F 2 "" H 4600 1500 50  0000 C CNN
 F 3 "" H 4600 1500 50  0000 C CNN
@@
 L R_Small R36
 U 1 1 58B2ED89
-P 7350 2050
-F 0 "R36" H 7380 2070 50  0000 L CNN
-F 1 "0/DNP" H 7380 2010 50  0000 L CNN
-F 2 "" H 7350 2050 50  0000 C CNN
-F 3 "" H 7350 2050 50  0000 C CNN
-	1    7350 2050
+P 7900 2050
+F 0 "R36" H 7930 2070 50  0000 L CNN
+F 1 "0/DNP" H 7930 2010 50  0000 L CNN
+F 2 "" H 7900 2050 50  0000 C CNN
+F 3 "" H 7900 2050 50  0000 C CNN
+	1    7900 2050
 	1    0    0    -1
 $EndComp
@@
 L C_Small C27
 U 1 1 58B2F002
-P 7350 2350
-F 0 "C27" H 7360 2420 50  0000 L CNN
-F 1 "10uF/6.3V" H 7360 2270 50  0000 L CNN
-F 2 "" H 7350 2350 50  0000 C CNN
-F 3 "" H 7350 2350 50  0000 C CNN
-	1    7350 2350
+P 7900 2350
+F 0 "C27" H 7910 2420 50  0000 L CNN
+F 1 "10uF/6.3V" H 7910 2270 50  0000 L CNN
+F 2 "" H 7900 2350 50  0000 C CNN
+F 3 "" H 7900 2350 50  0000 C CNN
+	1    7900 2350
 	1    0    0    -1
 $EndComp
@@
 L GND #PWR010
 U 1 1 58B2F008
-P 7350 2500
-F 0 "#PWR010" H 7350 2250 50  0001 C CNN
-F 1 "GND" H 7350 2350 50  0000 C CNN
-F 2 "" H 7350 2500 50  0000 C CNN
-F 3 "" H 7350 2500 50  0000 C CNN
-	1    7350 2500
+P 7900 2500
+F 0 "#PWR010" H 7900 2250 50  0001 C CNN
+F 1 "GND" H 7900 2350 50  0000 C CNN
+F 2 "" H 7900 2500 50  0000 C CNN
+F 3 "" H 7900 2500 50  0000 C CNN
+	1    7900 2500
 	1    0    0    -1
 $EndComp
@@
 L +VSOURCE #PWR011
 U 1 1 58B2F270
-P 7350 1900
-F 0 "#PWR011" H 7350 1750 50  0001 C CNN
-F 1 "+VSOURCE" H 7350 2040 50  0000 C CNN
-F 2 "" H 7350 1900 50  0000 C CNN
-F 3 "" H 7350 1900 50  0000 C CNN
-	1    7350 1900
+P 7900 1900
+F 0 "#PWR011" H 7900 1750 50  0001 C CNN
+F 1 "+VSOURCE" H 7900 2040 50  0000 C CNN
+F 2 "" H 7900 1900 50  0000 C CNN
+F 3 "" H 7900 1900 50  0000 C CNN
+	1    7900 1900
 	1    0    0    -1
 $EndComp
@@
 P 3275 4900
 F 0 "C41" H 3285 4970 50  0000 L CNN
-F 1 "4.7uF/50V" H 3285 4820 50  0000 L CNN
+F 1 "10uF/6.3V" H 3285 4820 50  0000 L CNN
 F 2 "" H 3275 4900 50  0000 C CNN
 F 3 "" H 3275 4900 50  0000 C CNN
@@
 	5800 2825 5600 2825
 Wire Wire Line
-	5600 2825 5600 3325
+	5600 2600 5600 3325
 Wire Wire Line
 	5275 2550 5275 2450
@@
 Connection ~ 4600 1650
 Wire Wire Line
-	7050 2200 7350 2200
-Wire Wire Line
-	7350 2450 7350 2500
-Wire Wire Line
-	7350 2150 7350 2250
-Connection ~ 7350 2200
-Wire Wire Line
-	7350 1900 7350 1950
+	7050 2200 7900 2200
+Wire Wire Line
+	7900 2450 7900 2500
+Wire Wire Line
+	7900 2150 7900 2250
+Connection ~ 7900 2200
+Wire Wire Line
+	7900 1900 7900 1950
 Wire Wire Line
 	3625 3675 3625 3725
@@
 	1    0    0    -1
 $EndComp
+Wire Wire Line
+	5600 2600 5925 2600
+Wire Wire Line
+	5925 2600 5925 2200
+Connection ~ 5925 2200
+Connection ~ 5600 2825
+Text Label 3300 4575 0    60   ~ 0
+PMICB_VSOURCE
+Text Label 7125 2200 0    60   ~ 0
+PMICB_VSOURCE
+Text Label 5400 6050 0    60   ~ 0
+PMICB_EPAD
+Text Label 4200 1350 0    60   ~ 0
+PMICB_VPOS
+Text Label 5550 5400 0    60   ~ 0
+PMICB_VSOURCE
+Text Label 6600 4650 0    60   ~ 0
+PMICB_EPAD
 $EndSCHEMATC

Commit message: update sch
Connections:
- wire segments 195 -> 194
Changed lines of the file:
@@
 	1050 3750 1050 3800
 Wire Wire Line
-	3700 4050 1050 4050
+	1050 4050 4075 4050
 Wire Wire Line
 	3700 5000 3700 5050
@@
 	1525 4225 1525 4050
 Connection ~ 1525 4050
-Wire Wire Line
-	3725 4050 4075 4050
 Wire Wire Line
 	2725 4725 4075 4725
@@
 Text Label 6600 4650 0    60   ~ 0
 PMICB_EPAD
+Text Label 3525 4125 0    60   ~ 0
+PMICB_EPAD
+Text Label 4925 6250 1    60   ~ 0
+PMICB_EPAD
 $EndSCHEMATC

Commit message: update sch
Parts:
- added C1: 10uF/25V, Capacitors_Tantalum_SMD:TantalC_SizeB_EIA-3528_HandSoldering, symbol CP1_Small
- added C2: 10uF, symbol C_Small
- added P1: USB_OTG, symbol USB_OTG
- added U2: NCP1117ST33T3G, TO_SOT_Packages_SMD:SOT-223, symbol NCP1117ST33T3G
Connections:
- net +3V15: now also C2.1, U2.2 (VO)
- net +VSOURCE: now also C1.1, P1.1 (VBUS), U2.3 (VI)
- net GND: now also C1.2, C2.2, P1.5 (GND), P1.6 (shield), U2.1 (GND)
- no-connect marks 5 -> 8
Changed lines of the file:
@@
 Text Label 4925 6250 1    60   ~ 0
 PMICB_EPAD
+$Comp
+L USB_OTG P1
+U 1 1 58B48648
+P 1175 1350
+F 0 "P1" H 1500 1225 50  0000 C CNN
+F 1 "USB_OTG" H 1175 1550 50  0000 C CNN
+F 2 "" V 1125 1250 50  0000 C CNN
+F 3 "" V 1125 1250 50  0000 C CNN
+	1    1175 1350
+	0    -1   1    0
+$EndComp
+$Comp
+L +VSOURCE #PWR036
+U 1 1 58B48D51
+P 1750 1075
+F 0 "#PWR036" H 1750 925 50  0001 C CNN
+F 1 "+VSOURCE" H 1750 1215 50  0000 C CNN
+F 2 "" H 1750 1075 50  0000 C CNN
+F 3 "" H 1750 1075 50  0000 C CNN
+	1    1750 1075
+	1    0    0    -1
+$EndComp
+NoConn ~ 1475 1250
+NoConn ~ 1475 1350
+NoConn ~ 1475 1450
+Wire Wire Line
+	1475 1550 1525 1550
+Wire Wire Line
+	1525 1550 1525 1800
+Wire Wire Line
+	1525 1800 1075 1800
+Wire Wire Line
+	1075 1750 1075 1850
+$Comp
+L GND #PWR037
+U 1 1 58B493F5
+P 1075 1850
+F 0 "#PWR037" H 1075 1600 50  0001 C CNN
+F 1 "GND" H 1075 1700 50  0000 C CNN
+F 2 "" H 1075 1850 50  0000 C CNN
+F 3 "" H 1075 1850 50  0000 C CNN
+	1    1075 1850
+	1    0    0    -1
+$EndComp
+Connection ~ 1075 1800
+Wire Wire Line
+	1475 1150 1750 1150
+Wire Wire Line
+	1750 1150 1750 1075
+$Comp
+L NCP1117ST33T3G U2
+U 1 1 58B498CB
+P 1900 2550
+F 0 "U2" H 1900 2775 50  0000 C CNN
+F 1 "NCP1117ST33T3G" H 1900 2700 50  0000 C CNN
+F 2 "TO_SOT_Packages_SMD:SOT-223" H 1950 2300 50  0001 L CNN
+F 3 "" H 1900 2550 50  0000 C CNN
+	1    1900 2550
+	1    0    0    -1
+$EndComp
+$Comp
+L +VSOURCE #PWR038
+U 1 1 58B49FF1
+P 1350 2400
+F 0 "#PWR038" H 1350 2250 50  0001 C CNN
+F 1 "+VSOURCE" H 1350 2540 50  0000 C CNN
+F 2 "" H 1350 2400 50  0000 C CNN
+F 3 "" H 1350 2400 50  0000 C CNN
+	1    1350 2400
+	1    0    0    -1
+$EndComp
+$Comp
+L CP1_Small C1
+U 1 1 58B4A250
+P 1350 2775
+F 0 "C1" H 1360 2845 50  0000 L CNN
+F 1 "10uF/25V" H 1360 2695 50  0000 L CNN
+F 2 "Capacitors_Tantalum_SMD:TantalC_SizeB_EIA-3528_HandSoldering" H 1350 2775 50  0000 C CNN
+F 3 "" H 1350 2775 50  0000 C CNN
+	1    1350 2775
+	1    0    0    -1
+$EndComp
+$Comp
+L C_Small C2
+U 1 1 58B4A4AB
+P 2350 2775
+F 0 "C2" H 2360 2845 50  0000 L CNN
+F 1 "10uF" H 2360 2695 50  0000 L CNN
+F 2 "" H 2350 2775 50  0000 C CNN
+F 3 "" H 2350 2775 50  0000 C CNN
+	1    2350 2775
+	1    0    0    -1
+$EndComp
+$Comp
+L +3V15 #PWR039
+U 1 1 58B4A5F0
+P 2450 2400
+F 0 "#PWR039" H 2450 2250 50  0001 C CNN
+F 1 "+3V15" H 2450 2540 50  0000 C CNN
+F 2 "" H 2450 2400 50  0000 C CNN
+F 3 "" H 2450 2400 50  0000 C CNN
+	1    2450 2400
+	1    0    0    -1
+$EndComp
+$Comp
+L GND #PWR040
+U 1 1 58B4A74F
+P 1350 2950
+F 0 "#PWR040" H 1350 2700 50  0001 C CNN
+F 1 "GND" H 1350 2800 50  0000 C CNN
+F 2 "" H 1350 2950 50  0000 C CNN
+F 3 "" H 1350 2950 50  0000 C CNN
+	1    1350 2950
+	1    0    0    -1
+$EndComp
+$Comp
+L GND #PWR041
+U 1 1 58B4A826
+P 1900 2950
+F 0 "#PWR041" H 1900 2700 50  0001 C CNN
+F 1 "GND" H 1900 2800 50  0000 C CNN
+F 2 "" H 1900 2950 50  0000 C CNN
+F 3 "" H 1900 2950 50  0000 C CNN
+	1    1900 2950
+	1    0    0    -1
+$EndComp
+$Comp
+L GND #PWR042
+U 1 1 58B4A8FD
+P 2350 2950
+F 0 "#PWR042" H 2350 2700 50  0001 C CNN
+F 1 "GND" H 2350 2800 50  0000 C CNN
+F 2 "" H 2350 2950 50  0000 C CNN
+F 3 "" H 2350 2950 50  0000 C CNN
+	1    2350 2950
+	1    0    0    -1
+$EndComp
+Wire Wire Line
+	1900 2850 1900 2950
+Wire Wire Line
+	1350 2875 1350 2950
+Wire Wire Line
+	1350 2400 1350 2675
+Wire Wire Line
+	1600 2550 1350 2550
+Connection ~ 1350 2550
+Wire Wire Line
+	2200 2550 2450 2550
+Wire Wire Line
+	2450 2550 2450 2400
+Wire Wire Line
+	2350 2675 2350 2550
+Connection ~ 2350 2550
+Wire Wire Line
+	2350 2875 2350 2950
 $EndSCHEMATC

Commit message: update sch
Parts:
- added P2: CONN_01X06, symbol CONN_01X06
Connections:
- net +15V(EINK): now also P2.3 (P3)
- net +22V(EINK): now also P2.2 (P2)
- net +3V15(EINK): now also P2.4 (P4)
- net -1V25(EINK): now also P2.5 (P5)
- net -20V(EINK): now also P2.1 (P1)
- net GND: now also P2.6 (P6)
Changed lines of the file:
@@
 Wire Wire Line
 	2350 2875 2350 2950
+$Comp
+L CONN_01X06 P2
+U 1 1 58B4D35A
+P 1550 6275
+F 0 "P2" H 1550 6625 50  0000 C CNN
+F 1 "CONN_01X06" V 1650 6275 50  0000 C CNN
+F 2 "" H 1550 6275 50  0000 C CNN
+F 3 "" H 1550 6275 50  0000 C CNN
+	1    1550 6275
+	-1   0    0    -1
+$EndComp
+$Comp
+L -20V(EINK) #PWR?
+U 1 1 58B4D943
+P 1900 5950
+F 0 "#PWR?" H 1900 5800 50  0001 C CNN
+F 1 "-20V(EINK)" H 1900 6090 50  0000 C CNN
+F 2 "" H 1900 5950 50  0000 C CNN
+F 3 "" H 1900 5950 50  0000 C CNN
+	1    1900 5950
+	1    0    0    -1
+$EndComp
+$Comp
+L +22V(EINK) #PWR?
+U 1 1 58B4D9E1
+P 2350 5950
+F 0 "#PWR?" H 2350 5800 50  0001 C CNN
+F 1 "+22V(EINK)" H 2350 6090 50  0000 C CNN
+F 2 "" H 2350 5950 50  0000 C CNN
+F 3 "" H 2350 5950 50  0000 C CNN
+	1    2350 5950
+	1    0    0    -1
+$EndComp
+$Comp
+L +15V(EINK) #PWR?
+U 1 1 58B4DA7F
+P 2800 5950
+F 0 "#PWR?" H 2800 5800 50  0001 C CNN
+F 1 "+15V(EINK)" H 2800 6090 50  0000 C CNN
+F 2 "" H 2800 5950 50  0000 C CNN
+F 3 "" H 2800 5950 50  0000 C CNN
+	1    2800 5950
+	1    0    0    -1
+$EndComp
+$Comp
+L +3V15(EINK) #PWR?
+U 1 1 58B4DC31
+P 2125 6175
+F 0 "#PWR?" H 2125 6025 50  0001 C CNN
+F 1 "+3V15(EINK)" H 2125 6315 50  0000 C CNN
+F 2 "" H 2125 6175 50  0000 C CNN
+F 3 "" H 2125 6175 50  0000 C CNN
+	1    2125 6175
+	1    0    0    -1
+$EndComp
+$Comp
+L -1V25(EINK) #PWR?
+U 1 1 58B4DCCF
+P 2625 6175
+F 0 "#PWR?" H 2625 6025 50  0001 C CNN
+F 1 "-1V25(EINK)" H 2625 6315 50  0000 C CNN
+F 2 "" H 2625 6175 50  0000 C CNN
+F 3 "" H 2625 6175 50  0000 C CNN
+	1    2625 6175
+	1    0    0    -1
+$EndComp
+$Comp
+L GND #PWR?
+U 1 1 58B4DDB0
+P 1900 6650
+F 0 "#PWR?" H 1900 6400 50  0001 C CNN
+F 1 "GND" H 1900 6500 50  0000 C CNN
+F 2 "" H 1900 6650 50  0000 C CNN
+F 3 "" H 1900 6650 50  0000 C CNN
+	1    1900 6650
+	1    0    0    -1
+$EndComp
+Wire Wire Line
+	1750 6025 1900 6025
+Wire Wire Line
+	1900 6025 1900 5950
+Wire Wire Line
+	1750 6125 2350 6125
+Wire Wire Line
+	2350 6125 2350 5950
+Wire Wire Line
+	1750 6225 2800 6225
+Wire Wire Line
+	2800 6225 2800 5950
+Wire Wire Line
+	1750 6325 2125 6325
+Wire Wire Line
+	2125 6325 2125 6175
+Wire Wire Line
+	1750 6425 2625 6425
+Wire Wire Line
+	2625 6425 2625 6175
+Wire Wire Line
+	1750 6525 1900 6525
+Wire Wire Line
+	1900 6525 1900 6650
 $EndSCHEMATC

Commit message: update sch
Parts:
- removed P2: CONN_01X06, symbol CONN_01X06
- added P2: CONN_01X09, symbol CONN_01X09
- added P3: CONN_01X05, symbol CONN_01X05
- added P4: CONN_01X02, symbol CONN_01X02
- added P5: 3V3, symbol CONN_01X01
Connections:
- net labels added: -15V(EINK)
- wire segments 220 -> 233
