File: einkpmic.sch (KiCad schematic (older format))
At the start: 72 parts, among them P1 USB_OTG, P2 CONN_01X09, P3 CONN_01X05, P4 CONN_01X02, P5 3V3, U1 TPS65185, U2 NCP1117ST33T3G

Commit message: update sch
Parts:
- removed P3: CONN_01X05, symbol CONN_01X05
- added P3: CONN_01X08, symbol CONN_01X08
Connections:
- wire segments 233 -> 237
Changed lines of the file:
@@
 Text Label 1350 7000 0    60   ~ 0
 PMIC_PGOOD
-$Comp
-L CONN_01X05 P3
-U 1 1 58B55BC4
-P 1000 6800
-F 0 "P3" H 1000 7100 50  0000 C CNN
-F 1 "CONN_01X05" V 1100 6800 50  0000 C CNN
-F 2 "" H 1000 6800 50  0000 C CNN
-F 3 "" H 1000 6800 50  0000 C CNN
-	1    1000 6800
-	-1   0    0    -1
-$EndComp
 Wire Wire Line
 	1200 6600 2200 6600
@@
 	1    0    0    -1
 $EndComp
+Text Label 1350 7100 0    60   ~ 0
+I2C1_SDA
+Text Label 1350 7200 0    60   ~ 0
+I2C1_SCL
+$Comp
+L GND #PWR?
+U 1 1 58B5A5E8
+P 1350 7375
+F 0 "#PWR?" H 1350 7125 50  0001 C CNN
+F 1 "GND" H 1350 7225 50  0000 C CNN
+F 2 "" H 1350 7375 50  0000 C CNN
+F 3 "" H 1350 7375 50  0000 C CNN
+	1    1350 7375
+	1    0    0    -1
+$EndComp
+$Comp
+L CONN_01X08 P3
+U 1 1 58B5A6CD
+P 1000 6950
+F 0 "P3" H 1000 7400 50  0000 C CNN
+F 1 "CONN_01X08" V 1100 6950 50  0000 C CNN
+F 2 "" H 1000 6950 50  0000 C CNN
+F 3 "" H 1000 6950 50  0000 C CNN
+	1    1000 6950
+	-1   0    0    -1
+$EndComp
+Wire Wire Line
+	1200 7100 2200 7100
+Wire Wire Line
+	1200 7200 2200 7200
+Wire Wire Line
+	1200 7300 1350 7300
+Wire Wire Line
+	1350 7300 1350 7375
 $EndSCHEMATC

Commit message: update footprint
Parts:
- C1: footprint Capacitors_Tantalum_SMD:TantalC_SizeB_EIA-3528_HandSoldering -> Capacitors_Tantalum_SMD:Tantalum_Case-B_EIA-3528-21_Hand
- C2, C23, C24, C25, C26, C27, C28, C29, C30, C31, C32, C33, C34, C35, C36, C37, C38, C39, C41, C42, C44, C45: footprint (none) -> Capacitors_SMD:C_0603_HandSoldering
- D10, D5, D6, D7, D8, D9: footprint (none) -> Diodes_SMD:SOD-123
- L3, L4: footprint (none) -> Inductors:Inductor_Taiyo-Yuden_NR-50xx_HandSoldering
- P1: footprint (none) -> SmartEye:USB_Micro-B
- P2: footprint (none) -> Connectors:CONN_2.54mm_1x9
- P3: footprint (none) -> Connectors:CONN_2.54mm_1x8
- P4: footprint (none) -> Connectors:CONN_2.54mm_1x2
- P5: footprint (none) -> Connectors:CONN_2.54mm_1x1
- R253, R33, R34, R35, R36, R37, R38, R39, R40, R41, R42, R43, R44, R45, R46, R47, R48, R49, R50, R52, R53, R55, R57, R59, R60, R61, R63, R66, R67, RT1, SH35, SH37, SH38, SH39: footprint (none) -> Resistors_SMD:R_0603_HandSoldering
- U1: footprint (none) -> Housings_DFN_QFN:QFN-48-1EP_7x7mm_Pitch0.5mm

Commit message: update pcb
Changed lines of the file:
@@
 L -1V25(EINK) #PWR045
 U 1 1 58B4DCCF
-P 1575 5475
-F 0 "#PWR045" H 1575 5325 50  0001 C CNN
-F 1 "-1V25(EINK)" H 1575 5615 50  0000 C CNN
-F 2 "" H 1575 5475 50  0000 C CNN
-F 3 "" H 1575 5475 50  0000 C CNN
-	1    1575 5475
+P 2075 5475
+F 0 "#PWR045" H 2075 5325 50  0001 C CNN
+F 1 "-1V25(EINK)" H 2075 5615 50  0000 C CNN
+F 2 "" H 2075 5475 50  0000 C CNN
+F 3 "" H 2075 5475 50  0000 C CNN
+	1    2075 5475
 	1    0    0    -1
 $EndComp
@@
 L -15V(EINK) #PWR047
 U 1 1 58B522EA
-P 2075 5475
-F 0 "#PWR047" H 2075 5325 50  0001 C CNN
-F 1 "-15V(EINK)" H 2075 5615 50  0000 C CNN
-F 2 "" H 2075 5475 50  0000 C CNN
-F 3 "" H 2075 5475 50  0000 C CNN
-	1    2075 5475
+P 1575 5475
+F 0 "#PWR047" H 1575 5325 50  0001 C CNN
+F 1 "-15V(EINK)" H 1575 5615 50  0000 C CNN
+F 2 "" H 1575 5475 50  0000 C CNN
+F 3 "" H 1575 5475 50  0000 C CNN
+	1    1575 5475
 	1    0    0    -1
 $EndComp

Commit message: update
Parts:
- removed R253, SH35, SH37, SH38, SH39: 0/DNP, Resistors_SMD:R_0603_HandSoldering, symbol R_Small
- added P6: CONN_01X01, AirBox:thermal, symbol CONN_01X01
Connections:
- wire segments 237 -> 233
