File: einkpmic.kicad_pcb (KiCad board)
At the start: 2 copper layers, 72 parts, among them P1 USB_OTG, P2 CONN_01X09, P3 CONN_01X08, P4 CONN_01X02, P5 3V3, U1 TPS65185, U2 NCP1117ST33T3G

Commit message: update pcb
Parts:
- added REF**: thermal, einkpmic:thermal, B.Cu at (99.7, 80.8)
- moved P5 179.2 mm to (64.2, 70.7)
- moved C2 175.4 mm to (61.3, 71.7), turned to 270 degrees
- moved R45 159.7 mm to (72.6, 73.6), turned to 270 degrees
- moved R40 158.5 mm to (80.3, 74.2)
- moved R52 152.1 mm to (80.3, 83.7), turned to 180 degrees
- moved R57 149.9 mm to (80.5, 94.0), turned to 180 degrees
- moved RT1 148.4 mm to (85.3, 68.1), turned to 90 degrees
- moved R61 147.2 mm to (93.2, 92.7), turned to 270 degrees
- moved R60 145.7 mm to (91.6, 92.7), turned to 90 degrees
- moved C41 144.9 mm to (80.4, 89.6), turned to 180 degrees
- moved R41 140.7 mm to (80.3, 72.6), turned to 180 degrees
- moved SH35 139.8 mm to (80.4, 88.0), turned to 180 degrees
- moved R55 139.1 mm to (80.5, 92.4), turned to 180 degrees
- moved R50 138.9 mm to (80.3, 82.1), turned to 180 degrees
- moved R33 138.4 mm to (100.3, 68.1), turned to 90 degrees
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Connections:
- P2 pad 4: -1V25(EINK) -> -15V(EINK)
- P2 pad 5: -15V(EINK) -> -1V25(EINK)
Routing:
- net GND: track 0.00 -> 545.2 mm, vias 0 -> 11
- net /PMICB_EPAD: track 0.00 -> 107.7 mm
- net -20V(EINK): track 0.00 -> 107.1 mm
- net +VSOURCE: track 0.00 -> 80.6 mm, vias 0 -> 2
- net /PMICB_VSOURCE: track 0.00 -> 71.7 mm, vias 0 -> 3
- net +22V(EINK): track 0.00 -> 68.6 mm
- net +3V15: track 0.00 -> 65.5 mm, vias 0 -> 1
- net /E_PMIC_PWR0: track 0.00 -> 56.9 mm
- net -1V25(EINK): track 0.00 -> 54.0 mm
- net /PMIC_PGOOD: track 0.00 -> 53.0 mm
- net Net-(D10-Pad1): track 0.00 -> 44.9 mm
- net /I2C1_SDA: track 0.00 -> 40.5 mm
- net /PMICB_VPOS: track 0.00 -> 40.1 mm, vias 0 -> 2
- net Net-(R46-Pad1): track 0.00 -> 38.5 mm
- net /I2C1_SCL: track 0.00 -> 35.5 mm
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- added copper zone on B.Cu, net GND
- added copper zone on F.Cu, net GND
Other:
- board outline added: 100 x 40 mm
- net class Default: trace_width 0.25 -> 0.28
- net class POWER added: clearance 0.2, trace_width 0.8, via_dia 0.6, via_drill 0.4
- board text added: "EinkPMIC v0.1"

Commit message: update
Parts:
- removed R253, SH35, SH37, SH38, SH39: 0/DNP, Resistors_SMD:R_0603_HandSoldering
- moved D10 19.6 mm to (110.1, 89.0)
- moved C37 19.5 mm to (109.6, 84.3)
- moved C36 19.4 mm to (109.6, 86.1)
- moved C38 11.7 mm to (105.6, 86.1), turned to 0 degrees
- moved C41 11.4 mm to (91.0, 85.5)
- moved C33 10.6 mm to (91.0, 79.5)
- moved C44 8.77 mm to (101.9, 88.7)
- moved R59 7.79 mm to (104.7, 91.6)
- moved C29 7.43 mm to (107.4, 75.5), turned to 0 degrees
- moved R63 5.20 mm to (101.3, 92.8)
- moved C45 4.27 mm to (97.0, 88.7)
- moved R67 3.60 mm to (98.1, 92.8)
- moved R66 3.60 mm to (99.7, 92.8)
- moved R61 2.60 mm to (90.6, 92.6)
- moved C42 2.60 mm to (94.1, 92.7)
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Connections:
- U1 pad 14: Net-(SH39-Pad1) -> GND
- U1 pad 19: Net-(SH38-Pad2) -> /PMICB_VPOS
- U1 pad 29: Net-(R253-Pad2) -> Net-(C35-Pad1)
- U1 pad 35: Net-(SH37-Pad2) -> Net-(C30-Pad1)
- U1 pad 9: Net-(SH35-Pad1) -> Net-(C32-Pad1)
Routing:
- net Net-(C30-Pad1): track 20.7 -> 50.3 mm
- net Net-(C35-Pad1): track 23.2 -> 52.4 mm
- net GND: track 545.2 -> 516.3 mm, vias 11 -> 25
- net Net-(SH37-Pad2): track 27.8 -> 0.00 mm
- net Net-(R253-Pad2): track 25.8 -> 0.00 mm
- net Net-(C25-Pad1): track 22.4 -> 47.9 mm, vias 2 -> 0
- net +3V15: track 65.5 -> 42.0 mm, vias 1 -> 2
- net Net-(SH35-Pad1): track 17.3 -> 0.00 mm
- net Net-(C32-Pad1): track 31.8 -> 46.9 mm
- net Net-(SH39-Pad1): track 11.9 -> 0.00 mm
- net Net-(SH38-Pad2): track 11.4 -> 0.00 mm
- net /PMIC_PGOOD: track 53.0 -> 44.0 mm
- net Net-(R59-Pad2): track 15.6 -> 7.44 mm, vias 0 -> 2
- net /E_PMIC_PWR0: track 56.9 -> 61.7 mm
- net /I2C1_SDA: track 40.5 -> 35.9 mm
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Other:
- net class vsource added: clearance 0.2, trace_width 0.6, via_dia 0.6, via_drill 0.4

Commit message: update PCB
Parts:
- removed REF**: thermal, einkpmic:thermal
- added P6: CONN_01X01, AirBox:thermal, B.Cu at (99.7, 80.8)
- moved P5 2.70 mm to (66.9, 70.7)
Routing:
- net Net-(C2-Pad1): track 15.0 -> 17.7 mm
Other:
- board text added: "-15V"
- board text added: "-1V25"
- board text added: "-20V"
- board text added: "15V"
- board text added: "22V"
- board text added: "3V15"
- board text added: "GND"
- board text added: "INT_B"
- board text added: "PGOOD"
- board text added: "PWR0"
- board text added: "SCL"
- board text added: "SDA"
- board text added: "VC_CTL"
- board text added: "WAKEUP"
Changed lines of the file:
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@@
 (kicad_pcb (version 4) (host pcbnew 4.0.5+dfsg1-4)
   (general
-    (links 162)
+    (links 163)
     (no_connects 0)
-    (area 46.625 59.924999 150.075001 100.075001)
+    (area 49.924999 59.924999 150.075001 100.075001)
     (thickness 1.6)
-    (drawings 5)
-    (tracks 876)
+    (drawings 22)
+    (tracks 878)
     (zones 0)
     (modules 68)
@@
     (35 F.Paste user)
     (36 B.SilkS user)
-    (37 F.SilkS user hide)
+    (37 F.SilkS user)
     (38 B.Mask user)
     (39 F.Mask user)
@@
     (uvia_min_size 0.2)
     (uvia_min_drill 0.1)
-    (pcb_text_width 0.3)
-    (pcb_text_size 1.5 1.5)
+    (pcb_text_width 0.15)
+    (pcb_text_size 1 1)
     (mod_edge_width 0.15)
     (mod_text_size 1 1)
@@
   )
   (module Connectors:CONN_2.54mm_1x1 (layer F.Cu)
-    (at 64.2 70.7)
+    (at 66.9 70.7)
     (fp_text reference P5 (at 2 0) (layer F.SilkS)
       (effects (font (size 1 1) (thickness 0.15)))
@@
     )
   )
-  (module einkpmic:thermal (layer B.Cu)
+  (module AirBox:thermal (layer B.Cu)
     (at 99.7 80.8)
-    (fp_text reference REF** (at -2.6 -3.4) (layer B.SilkS)
+    (fp_text reference P6 (at -2.6 -3.4) (layer B.SilkS)
       (effects (font (size 1 1) (thickness 0.15)) (justify mirror))
     )
-    (fp_text value thermal (at 3.3 -3.2) (layer B.Fab)
+    (fp_text value CONN_01X01 (at 3.3 -3.2) (layer B.Fab)
       (effects (font (size 1 1) (thickness 0.15)) (justify mirror))
     )
-    (pad 1 smd rect (at 0 0) (size 5 5) (layers B.Cu B.Paste B.Mask))
+    (pad 1 smd rect (at 0 0) (size 5 5) (layers B.Cu B.Paste B.Mask)
+      (net 13 /PMICB_EPAD))
+    (pad "" np_thru_hole circle (at 0 0) (size 0.5 0.5) (drill 0.5) (layers *.Cu *.Mask B.SilkS))
+    (pad "" np_thru_hole circle (at 2 2) (size 0.5 0.5) (drill 0.5) (layers *.Cu *.Mask B.SilkS))
+    (pad "" np_thru_hole circle (at 0 1) (size 0.5 0.5) (drill 0.5) (layers *.Cu *.Mask B.SilkS))
+    (pad "" np_thru_hole circle (at -2 2) (size 0.5 0.5) (drill 0.5) (layers *.Cu *.Mask B.SilkS))
+    (pad "" np_thru_hole circle (at -1 0) (size 0.5 0.5) (drill 0.5) (layers *.Cu *.Mask B.SilkS))
+    (pad "" np_thru_hole circle (at 1 0) (size 0.5 0.5) (drill 0.5) (layers *.Cu *.Mask B.SilkS))
+    (pad "" np_thru_hole circle (at 0 -1) (size 0.5 0.5) (drill 0.5) (layers *.Cu *.Mask B.SilkS))
+    (pad "" np_thru_hole circle (at -2 -2) (size 0.5 0.5) (drill 0.5) (layers *.Cu *.Mask B.SilkS))
+    (pad "" np_thru_hole circle (at 2 -2) (size 0.5 0.5) (drill 0.5) (layers *.Cu *.Mask B.SilkS))
+  )
+  (gr_text GND (at 71.9 92 90) (layer F.SilkS)
+    (effects (font (size 1 1) (thickness 0.15)))
+  )
+  (gr_text SCL (at 69.3 92.1 90) (layer F.SilkS)
+    (effects (font (size 1 1) (thickness 0.15)))
+  )
+  (gr_text SDA (at 66.8 92.1 90) (layer F.SilkS)
+    (effects (font (size 1 1) (thickness 0.15)))
+  )
+  (gr_text PGOOD (at 64.3 91 90) (layer F.SilkS)
+    (effects (font (size 1 1) (thickness 0.15)))
+  )
+  (gr_text VC_CTL (at 61.8 91 90) (layer F.SilkS)
+    (effects (font (size 1 1) (thickness 0.15)))
+  )
+  (gr_text WAKEUP (at 59.2 90.5 90) (layer F.SilkS)
+    (effects (font (size 1 1) (thickness 0.15)))
+  )
+  (gr_text INT_B (at 56.7 91.5 90) (layer F.SilkS)
+    (effects (font (size 1 1) (thickness 0.15)))
+  )
+  (gr_text PWR0 (at 54 91.4 90) (layer F.SilkS)
+    (effects (font (size 1 1) (thickness 0.15)))
+  )
+  (gr_text 22V (at 74.3 66.8 90) (layer F.SilkS)
+    (effects (font (size 1 1) (thickness 0.15)))
+  )
+  (gr_text 15V (at 71.7 66.8 90) (layer F.SilkS)
+    (effects (font (size 1 1) (thickness 0.15)))
+  )
+  (gr_text 3V15 (at 69.3 67.2 90) (layer F.SilkS)
+    (effects (font (size 1 1) (thickness 0.15)))
+  )
+  (gr_text -15V (at 66.7 67.4 90) (layer F.SilkS)
+    (effects (font (size 1 1) (thickness 0.15)))
+  )
+  (gr_text -1V25 (at 64.1 67.8 90) (layer F.SilkS)
+    (effects (font (size 1 1) (thickness 0.15)))
+  )
+  (gr_text -20V (at 61.7 67.5 90) (layer F.SilkS)
+    (effects (font (size 1 1) (thickness 0.15)))
+  )
+  (gr_text "GND\n" (at 59 67 90) (layer F.SilkS)
+    (effects (font (size 1 1) (thickness 0.15)))
+  )
+  (gr_text "GND\n" (at 56.4 67 90) (layer F.SilkS)
+    (effects (font (size 1 1) (thickness 0.15)))
+  )
+  (gr_text GND (at 53.7 67 90) (layer F.SilkS)
+    (effects (font (size 1 1) (thickness 0.15)))
   )
   (gr_text "EinkPMIC   v0.1" (at 143.3 61.3) (layer F.SilkS)
@@
   (segment (start 120.1944 65.5637) (end 111.4342 74.3239) (width 0.6) (layer B.Cu) (net 1))
   (segment (start 62.45 84.8) (end 65.3827 84.8) (width 0.6) (layer F.Cu) (net 1))
-  (segment (start 71.79 94.96096) (end 71.73904 94.96096) (width 0.28) (layer B.Cu) (net 2) (status C00000))
-  (segment (start 71.73904 94.96096) (end 69.8 96.9) (width 0.28) (layer B.Cu) (net 2) (status 400000))
+  (segment (start 71.79 94.96096) (end 71.73904 94.96096) (width 0.28) (layer B.Cu) (net 2))
+  (segment (start 71.73904 94.96096) (end 69.8 96.9) (width 0.28) (layer B.Cu) (net 2))
   (segment (start 69.8 96.9) (end 60.4 96.9) (width 0.28) (layer B.Cu) (net 2))
   (via (at 60.4 96.9) (size 0.6) (drill 0.4) (layers F.Cu B.Cu) (net 2))
-  (segment (start 58.92 64.06096) (end 58.93904 64.06096) (width 0.28) (layer B.Cu) (net 2) (status C00000))
-  (segment (start 58.93904 64.06096) (end 60.6 62.4) (width 0.28) (layer B.Cu) (net 2) (status 400000))
+  (segment (start 58.92 64.06096) (end 58.93904 64.06096) (width 0.28) (layer B.Cu) (net 2))
+  (segment (start 58.93904 64.06096) (end 60.6 62.4) (width 0.28) (layer B.Cu) (net 2))
   (via (at 68 62.4) (size 0.6) (drill 0.4) (layers F.Cu B.Cu) (net 2))
   (segment (start 60.6 62.4) (end 68 62.4) (width 0.28) (layer B.Cu) (net 2))
-  (segment (start 58.92 64.06096) (end 58.92 64.12) (width 0.28) (layer B.Cu) (net 2) (status C00000))
-  (segment (start 58.92 64.12) (end 61.9 67.1) (width 0.28) (layer B.Cu) (net 2) (status 400000))
+  (segment (start 58.92 64.06096) (end 58.92 64.12) (width 0.28) (layer B.Cu) (net 2))
+  (segment (start 58.92 64.12) (end 61.9 67.1) (width 0.28) (layer B.Cu) (net 2))
   (via (at 67.8 67.1) (size 0.6) (drill 0.4) (layers F.Cu B.Cu) (net 2))
   (segment (start 61.9 67.1) (end 67.8 67.1) (width 0.28) (layer B.Cu) (net 2))
-  (segment (start 58.92 64.06096) (end 58.92 63.88) (width 0.28) (layer B.Cu) (net 2) (status C00000))
+  (segment (start 58.92 64.06096) (end 58.92 63.88) (width 0.28) (layer B.Cu) (net 2))
   (segment (start 134.1 86.2) (end 129.1 86.2) (width 0.28) (layer B.Cu) (net 2))
   (via (at 134.1 86.2) (size 0.6) (drill 0.4) (layers F.Cu B.Cu) (net 2))
@@
   (via (at 131.8 75.5) (size 0.6) (drill 0.4) (layers F.Cu B.Cu) (net 2))
   (segment (start 134 77.7) (end 131.8 75.5) (width 0.28) (layer B.Cu) (net 2))
-  (segment (start 140.5 85.1) (end 140.5 86.3) (width 0.28) (layer F.Cu) (net 2) (status 400000))
+  (segment (start 140.5 85.1) (end 140.5 86.3) (width 0.28) (layer F.Cu) (net 2))
   (segment (start 140.1 86.7) (end 140.1 86.9) (width 0.28) (layer B.Cu) (net 2))
   (via (at 140.1 86.7) (size 0.6) (drill 0.4) (layers F.Cu B.Cu) (net 2))
@@
   (via (at 83.3 76.4) (size 0.6) (drill 0.4) (layers F.Cu B.Cu) (net 2))
   (segment (start 82.1 77.6) (end 83.3 76.4) (width 0.28) (layer B.Cu) (net 2))
-  (segment (start 66.75 86.9) (end 69.7 86.9) (width 0.28) (layer F.Cu) (net 2) (status 400000))
+  (segment (start 66.75 86.9) (end 69.7 86.9) (width 0.28) (layer F.Cu) (net 2))
   (segment (start 69.7 86.9) (end 69.8 86.9) (width 0.28) (layer B.Cu) (net 2))
   (via (at 69.7 86.9) (size 0.6) (drill 0.4) (layers F.Cu B.Cu) (net 2))
@@
   (segment (start 123.7315 81.0236) (end 124.3982 81.6903) (width 0.28) (layer F.Cu) (net 2))
   (segment (start 107.1925 81.0236) (end 123.7315 81.0236) (width 0.28) (layer F.Cu) (net 2))
+  (segment (start 66.9 70.7) (end 65.912172 70.7) (width 0.28) (layer F.Cu) (net 3))
+  (segment (start 65.912172 70.7) (end 65.862172 70.75) (width 0.28) (layer F.Cu) (net 3))
+  (segment (start 65.862172 70.75) (end 64.2 70.75) (width 0.28) (layer F.Cu) (net 3))
   (segment (start 61.3 70.75) (end 62.0153 70.75) (width 0.28) (layer F.Cu) (net 3))
   (segment (start 64.2 70.75) (end 62.0153 70.75) (width 0.28) (layer F.Cu) (net 3))
-  (segment (start 64.2 70.7) (end 64.2 70.75) (width 0.28) (layer F.Cu) (net 3))
   (segment (start 62.6403 78.9097) (end 61.55 78.9097) (width 0.28) (layer F.Cu) (net 3))
   (segment (start 65.4873 76.0627) (end 62.6403 78.9097) (width 0.28) (layer F.Cu) (net 3))
